File: pyroDirector/igniter.kicad_sch (KiCad schematic)
At the start: 13 parts, among them J24 LED_ext, J25 Screw_Terminal_01x02, K3 PR12-5V-360-1C, Q12 MMBT2222A 1P, Q13 IRLB8721PbF

Commit message: Manufactured 2021-02-25
Parts:
- C4: LCSC (none) -> C49678
- D3: value SM4007 -> M7; LCSC (none) -> C95872
- Q12: LCSC (none) -> C8512
- R25: LCSC (none) -> C17673
- R26, R28, R30: LCSC (none) -> C17514
- R27: LCSC (none) -> C17408
- R29: LCSC (none) -> C17713
Changed lines of the file:
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@@
+      (effects (font (size 1.27 1.27)) hide)
+    )
+    (property "LCSC" "C17673" (id 4) (at 110.49 107.95 90)
       (effects (font (size 1.27 1.27)) hide)
     )
@@
       (effects (font (size 1.27 1.27)) (justify left) hide)
     )
+    (property "LCSC" "C8512" (id 4) (at 121.92 107.95 0)
+      (effects (font (size 1.27 1.27)) hide)
+    )
     (pin "1")
     (pin "2")
@@
     )
     (property "Datasheet" "~" (id 3) (at 147.32 128.27 0)
+      (effects (font (size 1.27 1.27)) hide)
+    )
+    (property "LCSC" "C17713" (id 4) (at 147.32 128.27 90)
       (effects (font (size 1.27 1.27)) hide)
     )
@@
       (effects (font (size 1.27 1.27)) hide)
     )
+    (property "LCSC" "C17514" (id 4) (at 180.34 121.92 0)
+      (effects (font (size 1.27 1.27)) hide)
+    )
     (pin "1")
     (pin "2")
@@
     )
     (property "Datasheet" "~" (id 3) (at 180.34 133.35 0)
+      (effects (font (size 1.27 1.27)) hide)
+    )
+    (property "LCSC" "C17514" (id 4) (at 180.34 133.35 0)
       (effects (font (size 1.27 1.27)) hide)
     )
@@
       (effects (font (size 1.27 1.27)) hide)
     )
+    (property "LCSC" "C17408" (id 4) (at 133.35 121.92 90)
+      (effects (font (size 1.27 1.27)) hide)
+    )
     (pin "1")
     (pin "2")
@@
       (effects (font (size 1.27 1.27)) hide)
     )
+    (property "LCSC" "C49678" (id 4) (at 190.5 133.35 0)
+      (effects (font (size 1.27 1.27)) hide)
+    )
     (pin "1")
     (pin "2")
@@
       (effects (font (size 1.27 1.27)) hide)
     )
+    (property "LCSC" "C17514" (id 4) (at 180.34 111.76 0)
+      (effects (font (size 1.27 1.27)) hide)
+    )
     (pin "1")
     (pin "2")
@@
       (effects (font (size 1.27 1.27)) (justify left))
     )
-    (property "Value" "SM4007" (id 1) (at 127 99.0599 90)
+    (property "Value" "M7" (id 1) (at 127 99.0599 90)
       (effects (font (size 1.27 1.27)) (justify left))
     )
@@
       (effects (font (size 1.27 1.27)) hide)
     )
+    (property "LCSC" "C95872" (id 4) (at 124.46 97.79 0)
+      (effects (font (size 1.27 1.27)) hide)
+    )
