File: input-panel/input-panel.kicad_sch (KiCad schematic)
At the start: 11 parts, among them J1 Conn_01x07_Male

Commit message: re-designed input panel PCB
Parts:
- S1, S2, S3, S4, S5, S6: footprint TL1105:SW_TL1105DF160Q -> SW_TL1105DF160Q
Changed lines of the file:
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@@
       (effects (font (size 1.27 1.27)) (justify right))
     )
-    (property "Footprint" "TL1105:SW_TL1105DF160Q" (id 2) (at 162.56 91.44 0)
+    (property "Footprint" "SW_TL1105DF160Q" (id 2) (at 162.56 91.44 0)
       (effects (font (size 1.27 1.27)) (justify bottom) hide)
     )
@@
       (effects (font (size 1.27 1.27)) (justify right))
     )
-    (property "Footprint" "TL1105:SW_TL1105DF160Q" (id 2) (at 187.96 91.44 0)
+    (property "Footprint" "SW_TL1105DF160Q" (id 2) (at 187.96 91.44 0)
       (effects (font (size 1.27 1.27)) (justify bottom) hide)
     )
@@
       (effects (font (size 1.27 1.27)) (justify right))
     )
-    (property "Footprint" "TL1105:SW_TL1105DF160Q" (id 2) (at 86.36 91.44 0)
+    (property "Footprint" "SW_TL1105DF160Q" (id 2) (at 86.36 91.44 0)
       (effects (font (size 1.27 1.27)) (justify bottom) hide)
     )
@@
       (effects (font (size 1.27 1.27)) (justify right))
     )
-    (property "Footprint" "TL1105:SW_TL1105DF160Q" (id 2) (at 213.36 91.44 0)
+    (property "Footprint" "SW_TL1105DF160Q" (id 2) (at 213.36 91.44 0)
       (effects (font (size 1.27 1.27)) (justify bottom) hide)
     )
@@
       (effects (font (size 1.27 1.27)) (justify right))
     )
-    (property "Footprint" "TL1105:SW_TL1105DF160Q" (id 2) (at 137.16 91.44 0)
+    (property "Footprint" "SW_TL1105DF160Q" (id 2) (at 137.16 91.44 0)
       (effects (font (size 1.27 1.27)) (justify bottom) hide)
     )
@@
       (effects (font (size 1.27 1.27)) (justify right))
     )
-    (property "Footprint" "TL1105:SW_TL1105DF160Q" (id 2) (at 111.76 91.44 0)
+    (property "Footprint" "SW_TL1105DF160Q" (id 2) (at 111.76 91.44 0)
       (effects (font (size 1.27 1.27)) (justify bottom) hide)
     )
@@
     )
     (path "/827fe059-08e0-48d9-8172-99e918124590"
-      (reference "S1") (unit 1) (value "BTN_CNCL") (footprint "TL1105:SW_TL1105DF160Q")
+      (reference "S1") (unit 1) (value "BTN_CNCL") (footprint "SW_TL1105DF160Q")
     )
     (path "/e3619dad-a23c-4f6e-8881-7188185a44b1"
-      (reference "S2") (unit 1) (value "BTN_DOWN") (footprint "TL1105:SW_TL1105DF160Q")
+      (reference "S2") (unit 1) (value "BTN_DOWN") (footprint "SW_TL1105DF160Q")
     )
     (path "/d07bde72-f89b-47ec-8ba2-5760048a78fb"
-      (reference "S3") (unit 1) (value "BTN_UP") (footprint "TL1105:SW_TL1105DF160Q")
+      (reference "S3") (unit 1) (value "BTN_UP") (footprint "SW_TL1105DF160Q")
     )
     (path "/263ef5a4-d43b-4d1e-801b-51643048d716"
-      (reference "S4") (unit 1) (value "BTN_LEFT") (footprint "TL1105:SW_TL1105DF160Q")
+      (reference "S4") (unit 1) (value "BTN_LEFT") (footprint "SW_TL1105DF160Q")
     )
     (path "/5a509bd6-3358-433f-83f1-fb48b9d5bc5a"
-      (reference "S5") (unit 1) (value "BTN_RIGHT") (footprint "TL1105:SW_TL1105DF160Q")
+      (reference "S5") (unit 1) (value "BTN_RIGHT") (footprint "SW_TL1105DF160Q")
     )
     (path "/844d3e0d-42ab-496b-bffa-a8a9ed2ba93d"
-      (reference "S6") (unit 1) (value "BTN_OK") (footprint "TL1105:SW_TL1105DF160Q")
-    )
-  )
+      (reference "S6") (unit 1) (value "BTN_OK") (footprint "SW_TL1105DF160Q")
+    )
+  )
